Commit message: documentation

File: xacro/dc_motor.xacro (robot description, xacro)
@@ -1,8 +1,7 @@
 <?xml version="1.0"?>
 <robot xmlns:xacro="http://www.ros.org/wiki/xacro">
-<!-- load parameters from yaml file -->
-<xacro:property name="params_yaml"  value="$(find gazebo_ros_motors)/params/dc_motor.yaml"/>
-<xacro:property name="motor_param" value="${load_yaml(params_yaml)}"/>
 <xacro:macro name="dc_motor" params="motor_name parent_link child_link *origin">
+  <!-- <xacro:property name="params_yaml" value="$(find gazebo_ros_motors)/params/dc_motor.yaml"/> -->
+  <xacro:property name="motor_param" value="${load_yaml(params_yaml)}"/>
   <joint name="${motor_name}" type="continuous">
       <parent link="${parent_link}"/>

File: xacro/joint_motor.xacro (robot description, xacro)
@@ -1,9 +1,7 @@
 <?xml version="1.0"?>
 <robot xmlns:xacro="http://www.ros.org/wiki/xacro">
-<!-- load parameters from yaml file -->
-<xacro:property name="params_yaml"  value="$(find gazebo_ros_motors)/params/joint_motor.yaml"/>
-<xacro:property name="motor_param" value="${load_yaml(params_yaml)}"/>
-<!-- ODE joint motor macro -->
 <xacro:macro name="joint_motor" params="motor_name parent_link child_link *origin">
+  <xacro:property name="params_yaml"  value="$(find gazebo_ros_motors)/params/joint_motor.yaml"/>
+  <xacro:property name="motor_param" value="${load_yaml(params_yaml)}"/>
   <joint name="${motor_name}" type="continuous">
       <parent link="${parent_link}"/>

File: xacro/test.xacro (robot description, xacro)
@@ -53,8 +53,10 @@
   <xacro:include filename="$(find gazebo_ros_motors)/xacro/dc_motor.xacro"/>
   <xacro:dc_motor motor_name="dc_motor" parent_link="base_link" child_link="wheel_link">
+    <xacro:property name="params_yaml" value="$(find gazebo_ros_motors)/params/dc_motor.yaml"/>
     <origin xyz="0 0 0.2" rpy="0 0 0"/>
   </xacro:dc_motor>
   <!-- <xacro:include filename="$(find gazebo_ros_motors)/xacro/joint_motor.xacro"/>
   <xacro:joint_motor motor_name="ode_motor" parent_link="base_link" child_link="wheel_link">
+    <xacro:property name="params_yaml" value="$(find gazebo_ros_motors)/params/joint_motor.yaml"/>
     <origin xyz="0 0 0.2" rpy="0 0 0"/>
   </xacro:joint_motor> -->

Commit message: joint state publishing fix

File: xacro/dc_motor.xacro (robot description, xacro)
@@ -35,4 +35,5 @@
       <gear_ratio>${motor_param['gear_ratio']}</gear_ratio>
       <encoder_ppr>${motor_param['encoder_ppr']}</encoder_ppr>
+      <rosDebugLevel>Debug</rosDebugLevel>
     </plugin>
   </gazebo>

File: xacro/joint_motor.xacro (robot description, xacro)
@@ -26,4 +26,5 @@
       <encoder_ppr>${motor_param['encoder_ppr']}</encoder_ppr>
       <encoder_to_shaft_ratio>${motor_param['encoder_to_shaft_ratio']}</encoder_to_shaft_ratio>
+      <rosDebugLevel>Debug</rosDebugLevel>
     </plugin>
   </gazebo>

File: xacro/test.xacro (robot description, xacro)
@@ -29,26 +29,40 @@
       <origin rpy="0 0 0" xyz="0 0 0"/>
   </joint>
-  <link name="wheel_link">
-    <visual>
-      <origin rpy="0 0 0" xyz="0 0 0"/>
-      <geometry>
-          <cylinder length="0.05" radius="0.11"/>
-      </geometry>
-    </visual>
-    <collision>
+  <xacro:macro name="wheel" params="name">
+    <link name="${name}_wheel_link">
+      <visual>
         <origin rpy="0 0 0" xyz="0 0 0"/>
         <geometry>
             <cylinder length="0.05" radius="0.11"/>
         </geometry>
-    </collision>
-    <inertial>
-      <origin rpy="0 0 0" xyz="0 0 0"/>
-      <geometry>
-          <cylinder length="0.05" radius="0.11"/>
-      </geometry>
-        <mass value="3.5"/>
-        <inertia ixx="0.0267" ixy="0" ixz="0" iyy="0.0267" iyz="0" izz="0.0506"/>
-    </inertial>
-  </link>
+      </visual>
+      <collision>
+          <origin rpy="0 0 0" xyz="0 0 0"/>
+          <geometry>
+              <cylinder length="0.05" radius="0.11"/>
+          </geometry>
+      </collision>
+      <inertial>
+        <origin rpy="0 0 0" xyz="0 0 0"/>
+        <geometry>
+            <cylinder length="0.05" radius="0.11"/>
+        </geometry>
+          <mass value="3.5"/>
+          <inertia ixx="0.0267" ixy="0" ixz="0" iyy="0.0267" iyz="0" izz="0.0506"/>
+      </inertial>
+    </link>
+  </xacro:macro>
+  <xacro:wheel name="one"/>
+  <xacro:wheel name="two"/>
+  <xacro:include filename="$(find gazebo_ros_motors)/xacro/joint_motor.xacro"/>
+  <xacro:joint_motor motor_name="one_motor" parent_link="base_link" child_link="one_wheel_link">
+    <xacro:property name="params_yaml" value="$(find gazebo_ros_motors)/params/joint_motor.yaml"/>
+    <origin xyz="0 0 0.2" rpy="0 0 0"/>
+  </xacro:joint_motor>
+  <xacro:joint_motor motor_name="two_motor" parent_link="base_link" child_link="two_wheel_link">
+    <xacro:property name="params_yaml" value="$(find gazebo_ros_motors)/params/joint_motor.yaml"/>
+    <origin xyz="0 0 0.4" rpy="0 0 0"/>
+  </xacro:joint_motor>
+  <!--
   <xacro:include filename="$(find gazebo_ros_motors)/xacro/dc_motor.xacro"/>
   <xacro:dc_motor motor_name="dc_motor" parent_link="base_link" child_link="wheel_link">
@@ -56,8 +70,4 @@
     <origin xyz="0 0 0.2" rpy="0 0 0"/>
   </xacro:dc_motor>
-  <!-- <xacro:include filename="$(find gazebo_ros_motors)/xacro/joint_motor.xacro"/>
-  <xacro:joint_motor motor_name="ode_motor" parent_link="base_link" child_link="wheel_link">
-    <xacro:property name="params_yaml" value="$(find gazebo_ros_motors)/params/joint_motor.yaml"/>
-    <origin xyz="0 0 0.2" rpy="0 0 0"/>
-  </xacro:joint_motor> -->
+  -->
 </robot>

Commit message: allow specifying axis

File: xacro/dc_motor.xacro (robot description, xacro)
@@ -1,5 +1,5 @@
 <?xml version="1.0"?>
 <robot xmlns:xacro="http://www.ros.org/wiki/xacro">
-<xacro:macro name="dc_motor" params="motor_name parent_link child_link *origin">
+<xacro:macro name="dc_motor" params="motor_name parent_link child_link *origin *axis">
   <!-- <xacro:property name="params_yaml" value="$(find gazebo_ros_motors)/params/dc_motor.yaml"/> -->
   <xacro:property name="motor_param" value="${load_yaml(params_yaml)}"/>
@@ -8,5 +8,6 @@
       <child link="${child_link}"/>
       <xacro:insert_block name="origin"/>
-      <axis xyz="0 0 1"/>
+      <xacro:insert_block name="axis"/>
+      <!-- <axis xyz="0 0 1"/> -->
       <dynamics damping="${motor_param['joint_damping']}" friction="${motor_param['joint_friction']}"/>
   </joint>
@@ -15,5 +16,5 @@
   </gazebo>
   <gazebo>
-    <plugin name="motor_plugin" filename="libgazebo_ros_dc_motor.so">
+    <plugin name="${motor_name}_plugin" filename="libgazebo_ros_dc_motor.so">
       <motor_shaft_joint>${motor_name}</motor_shaft_joint>
       <motor_wrench_frame>${child_link}</motor_wrench_frame>

Commit message: Update README

File: xacro/dc_motor.xacro (robot description, xacro)
@@ -9,5 +9,4 @@
       <xacro:insert_block name="origin"/>
       <xacro:insert_block name="axis"/>
-      <!-- <axis xyz="0 0 1"/> -->
       <dynamics damping="${motor_param['joint_damping']}" friction="${motor_param['joint_friction']}"/>
   </joint>

File: xacro/joint_motor.xacro (robot description, xacro)
@@ -1,5 +1,5 @@
 <?xml version="1.0"?>
 <robot xmlns:xacro="http://www.ros.org/wiki/xacro">
-<xacro:macro name="joint_motor" params="motor_name parent_link child_link *origin">
+<xacro:macro name="joint_motor" params="motor_name parent_link child_link *origin *axis">
   <xacro:property name="params_yaml"  value="$(find gazebo_ros_motors)/params/joint_motor.yaml"/>
   <xacro:property name="motor_param" value="${load_yaml(params_yaml)}"/>
@@ -8,5 +8,5 @@
       <child link="${child_link}"/>
       <xacro:insert_block name="origin"/>
-      <axis xyz="0 0 1"/>
+      <xacro:insert_block name="axis"/>
       <dynamics damping="${motor_param['joint_damping']}" friction="${motor_param['joint_friction']}"/>
   </joint>
