Commit message: Apply torque to joint, so it won't be misaligned with joint axis.

File: xacro/test.xacro (robot description, xacro)
@@ -68,4 +68,5 @@
     <xacro:property name="params_yaml" value="$(find gazebo_ros_motors)/params/dc_motor.yaml"/>
     <origin xyz="0 0 0.2" rpy="0 0 0"/>
+    <axis xyz="0 1 0" rpy="0 0 0"/>
   </xacro:dc_motor>
 </robot>
